File: Proyecto_Maletero.kicad_pcb (KiCad board)
At the start: 2 copper layers, 65.4 x 59.2 mm, 49 parts, among them J1 DE9_Pins, J2 Conn_01x02, J3 Conn_01x02, J4 Conn_01x03, J5 Conn_01x02, J6 DE9_Pins, J7 Conn_01x04, J9 Conn_01x04, K1 FINDER-34.51, Q2 MMBT5550L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

Commit message: Esquematico final y pasado al layout
Changed lines of the file:
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@@
 	(segment
 		(start 126.69521 116.194988)
-		(end 126.69521 116.145)
-		(width 0.4)
-		(layer "B.Cu")
-		(net 28)
-	)
-	(segment
-		(start 126.695222 116.195)
-		(end 126.69521 116.194988)
-		(width 0.4)
-		(layer "B.Cu")
-		(net 28)
-	)
-	(segment
-		(start 126.69521 116.145)
-		(end 126.695 116.14479)
-		(width 0.4)
-		(layer "B.Cu")
-		(net 28)
-	)
-	(segment
-		(start 126.695 116.14479)
-		(end 126.695 113.975)
+		(end 126.695222 116.195)
 		(width 0.4)
 		(layer "B.Cu")
@@
 		(width 0.4)
 		(layer "B.Cu")
+		(net 28)
+	)
+	(segment
+		(start 126.695 113.975)
+		(end 126.695 116.14479)
+		(width 0.4)
+		(layer "B.Cu")
+		(net 28)
+	)
+	(segment
+		(start 126.695 116.14479)
+		(end 126.69521 116.145)
+		(width 0.4)
+		(layer "B.Cu")
+		(net 28)
+	)
+	(segment
+		(start 126.69521 116.145)
+		(end 126.69521 116.194988)
+		(width 0.4)
+		(layer "B.Cu")
