File: Proyecto_Maletero/untitled.kicad_sch (KiCad schematic)
At the start: 31 parts, among them J2 Conn_01x02, J5 Conn_01x02, J7 Conn_01x04, J8 DE9_Pins, J9 Conn_01x04, K1 FINDER-34.51, Q2 MMBT5550L, SW1 SW_Push, SW2 SW_Push, U4 MCP2551-I-SN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

Commit message: Actualizacion layout
Colocacion idonias de tornillos, simetrias y reduccion de avisos de 8 a 2
Other:
- note added: "24.03.2025"
- note added: "AUTORS"
- note added: "Eric Trejo Sanchez Eloi Ortega Ortiz"
- note added: "Proyecto Maletero"
Changed lines of the file:
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@@
+		)
+	)
+	(text "AUTORS"
+		(exclude_from_sim no)
+		(at 181.61 168.402 0)
+		(effects
+			(font
+				(size 1.27 1.27)
+			)
+		)
+	)
+	(text "24.03.2025"
+		(exclude_from_sim no)
+		(at 207.264 193.04 0)
+		(effects
+			(font
+				(size 1.27 1.27)
+				(thickness 0.254)
+				(bold yes)
+			)
+			(justify left)
+		)
+	)
+	(text "Proyecto Maletero"
+		(exclude_from_sim no)
+		(at 186.944 189.738 0)
+		(effects
+			(font
+				(size 1.778 1.778)
+				(thickness 0.254)
+				(bold yes)
+			)
+			(justify left)
 		)
 	)
@@
 		)
 	)
+	(text "Eric Trejo Sanchez\nEloi Ortega Ortiz"
+		(exclude_from_sim no)
+		(at 177.546 173.736 0)
+		(effects
+			(font
+				(size 1.905 1.905)
+			)
+			(justify left)
+		)
+	)
