File: Proyecto_Maletero/untitled.kicad_sch (KiCad schematic)
At the start: 31 parts, among them J2 Conn_01x02, J5 Conn_01x02, J7 Conn_01x04, J8 DE9_Pins, J9 Conn_01x04, K1 FINDER-34.51, Q2 MMBT5550L, SW1 SW_Push, SW2 SW_Push, U4 MCP2551-I-SN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

Commit message: Version final final
Connections:
- net COLECTOR_RELE: now reaches D2.2 (A), K1.A2, Q2.3 (C)
- net RS: now reaches R11.2, U4.8 (Rs)
- net Analogico transistor renamed AN_TRANSISTOR
Changed lines of the file:
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@@
+		)
+	)
+	(global_label "COLECTOR_RELE"
+		(shape passive)
+		(at 231.14 60.96 180)
+		(fields_autoplaced yes)
+		(effects
+			(font
+				(size 1.27 1.27)
+			)
+			(justify right)
+		)
+		(property "Intersheetrefs" "${INTERSHEET_REFS}"
+			(at 214.5821 60.96 0)
+			(effects
+				(font
+					(size 1.27 1.27)
+				)
+				(justify right)
+				(hide yes)
+			)
+		)
+	)
+	(global_label "RS"
+		(shape passive)
+		(at 160.02 132.08 180)
+		(fields_autoplaced yes)
+		(effects
+			(font
+				(size 1.27 1.27)
+			)
+			(justify right)
+		)
+		(property "Intersheetrefs" "${INTERSHEET_REFS}"
+			(at 156.162 132.08 0)
+			(effects
+				(font
+					(size 1.27 1.27)
+				)
+				(justify right)
+				(hide yes)
+			)
 		)
 	)
@@
 		)
 	)
-	(global_label "Analogico transistor"
+	(global_label "AN_TRANSISTOR"
 		(shape passive)
 		(at 241.3 71.12 180)
@@
 		)
 		(property "Intersheetrefs" "${INTERSHEET_REFS}"
-			(at 220.6299 71.12 0)
+			(at 225.2862 71.12 0)
 			(effects
 				(font
@@
 		)
 		(property "Value" "10k"
-			(at 166.116 136.652 0)
-			(effects
-				(font
+			(at 165.1 136.652 0)
+			(effects
+				(font

Commit message: Ultimos cambios y revisiones
Changed lines of the file:
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@@
 		(on_board yes)
 		(dnp no)
-		(fields_autoplaced yes)
 		(property "Reference" "#PWR04"
 			(at 175.26 50.8 0)
@@
 		)
 		(property "Value" "GNDPWR"
-			(at 175.133 49.53 0)
+			(at 180.594 48.768 0)
 			(effects
 				(font
@@
 		(dnp no)
 		(property "Reference" "K1"
-			(at 257.81 49.5299 0)
+			(at 257.048 50.546 0)
 			(effects
 				(font
@@
 		(on_board yes)
 		(dnp no)
-		(fields_autoplaced yes)
 		(property "Reference" "#PWR038"
 			(at 227.33 50.8 0)
@@
 		)
 		(property "Value" "GNDPWR"
-			(at 227.203 49.53 0)
+			(at 221.488 49.53 0)
 			(effects
 				(font
@@
 		(on_board yes)
 		(dnp no)
-		(fields_autoplaced yes)
 		(property "Reference" "D2"
-			(at 233.68 49.5299 90)
+			(at 226.822 51.562 90)
 			(effects
 				(font
@@
 		)
 		(property "Value" "SM4001"
-			(at 233.68 52.0699 90)
-			(effects
-				(font
+			(at 227.584 54.102 90)
+			(effects
+				(font
