File: Proyecto_Maletero/_autosave-untitled.kicad_sch (KiCad schematic)
At the start: 31 parts, among them J2 Conn_01x02, J5 Conn_01x02, J7 Conn_01x04, J8 DE9_Pins, J9 Conn_01x04, K1 FINDER-34.51, Q2 MMBT5550L, SW1 SW_Push, SW2 SW_Push, U4 MCP2551-I-SN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

Commit message: Muchos arreglos de placement
Connections:
- net COLECTOR_RELE: now reaches D2.2 (A), K1.A2, Q2.3 (C)
- net Analogico transistor renamed AN_TRANSISTOR
Changed lines of the file:
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@@
+		)
+	)
+	(global_label "COLECTOR_RELE"
+		(shape passive)
+		(at 231.14 60.96 180)
+		(fields_autoplaced yes)
+		(effects
+			(font
+				(size 1.27 1.27)
+			)
+			(justify right)
+		)
+		(property "Intersheetrefs" "${INTERSHEET_REFS}"
+			(at 214.5821 60.96 0)
+			(effects
+				(font
+					(size 1.27 1.27)
+				)
+				(justify right)
+				(hide yes)
+			)
 		)
 	)
@@
 		)
 	)
-	(global_label "Analogico transistor"
+	(global_label "AN_TRANSISTOR"
 		(shape passive)
 		(at 241.3 71.12 180)
@@
 		)
 		(property "Intersheetrefs" "${INTERSHEET_REFS}"
-			(at 220.6299 71.12 0)
+			(at 225.2862 71.12 0)
 			(effects
 				(font
@@
 		)
 		(property "Value" "10k"
-			(at 166.116 136.652 0)
-			(effects
-				(font
+			(at 165.1 136.652 0)
+			(effects
+				(font
