File: Proyecto_Maletero/Proyecto_Maletero.kicad_pcb (KiCad board)
At the start: 2 copper layers, 65.6 x 60.1 mm, 49 parts, among them J1 DE9_Pins, J2 Conn_01x02, J3 Conn_01x02, J4 Conn_01x03, J5 Conn_01x02, J6 DE9_Pins, J7 Conn_01x04, J9 Conn_01x04, K1 FINDER-34.51, Q2 MMBT5550L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

Commit message: Muchos arreglos de placement
Parts:
- removed C13: 100n, Capacitor_SMD:C_0805_2012Metric
- removed J1: DE9_Pins, Connector_Dsub:DSUB-9_Pins_Horizontal_P2.77x2.54mm_EdgePinOffset9.40mm
- removed R6: 10k, Resistor_SMD:R_0805_2012Metric
- removed R7: 60, Resistor_SMD:R_0805_2012Metric
- removed U2: MCP2551-I-SN, Package_SO:SOIC-8_3.9x4.9mm_P1.27mm
- added C17: 100n, Capacitor_SMD:C_0805_2012Metric, F.Cu at (144.3, 102.0)
- added J8: DE9_Pins, Connector_Dsub:DSUB-9_Pins_Horizontal_P2.77x2.54mm_EdgePinOffset9.40mm, F.Cu at (162.5, 95.3)
- added R11: 10k, Resistor_SMD:R_0805_2012Metric, F.Cu at (151.9, 97.5)
- added R12: 60, Resistor_SMD:R_0805_2012Metric, F.Cu at (158.9, 98.3)
- added U4: MCP2551-I-SN, Package_SO:SOIC-8_3.9x4.9mm_P1.27mm, F.Cu at (149.8, 101.4)
- moved C14 7.36 mm to (151.0, 105.2), turned to 180 degrees
Connections:
- net Net-(D2-A) renamed COLECTOR_RELE
- net Net-(Q2-B) renamed AN_TRANSISTOR
Routing:
- net VBAT: track 0.31 -> 4.52 mm
- net Net-(U4-Rs): track 0.00 -> 3.10 mm
- net Net-(U2-Rs): track 3.10 -> 0.00 mm
- net CAN-: track 17.4 -> 19.1 mm

Commit message: Version final final
Connections:
- net Net-(U4-Rs) renamed RS
Changed lines of the file:
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@@
 	(net 48 "unconnected-(J8-Pad8)")
 	(net 49 "unconnected-(J8-Pad5)")
-	(net 50 "Net-(U4-Rs)")
-	(net 51 "unconnected-(U4-Vref-Pad5)")
-	(net 52 "AN_TRANSISTOR")
+	(net 50 "unconnected-(U4-Vref-Pad5)")
+	(net 51 "AN_TRANSISTOR")
+	(net 52 "RS")
 	(net 53 "COLECTOR_RELE")
 	(footprint "Resistor_SMD:R_0805_2012Metric"
@@
 		)
 		(property "Value" "DRV8870DDA"
-			(at 0 -0.145 0)
+			(at 0 -0.705 0)
 			(layer "F.Fab")
 			(effects
@@
 			(layers "F.Cu" "F.Mask" "F.Paste")
 			(roundrect_rratio 0.243902)
-			(net 52 "AN_TRANSISTOR")
+			(net 51 "AN_TRANSISTOR")
 			(pintype "passive")
 		)
@@
 			(layers "F.Cu" "F.Mask" "F.Paste")
 			(roundrect_rratio 0.243902)
-			(net 52 "AN_TRANSISTOR")
+			(net 51 "AN_TRANSISTOR")
 			(pintype "passive")
 		)
@@
 			(layers "F.Cu" "F.Mask" "F.Paste")
 			(roundrect_rratio 0.243902)
-			(net 50 "Net-(U4-Rs)")
+			(net 52 "RS")
 			(pintype "passive")
 		)
@@
 			(layers "F.Cu" "F.Mask" "F.Paste")
 			(roundrect_rratio 0.25)
-			(net 52 "AN_TRANSISTOR")
+			(net 51 "AN_TRANSISTOR")
 			(pinfunction "B")
 			(pintype "input")
@@
 			(layers "F.Cu" "F.Mask" "F.Paste")
 			(roundrect_rratio 0.25)
-			(net 51 "unconnected-(U4-Vref-Pad5)")
+			(net 50 "unconnected-(U4-Vref-Pad5)")
 			(pinfunction "Vref")
 			(pintype "power_out+no_connect")
@@
 			(layers "F.Cu" "F.Mask" "F.Paste")
 			(roundrect_rratio 0.25)
-			(net 50 "Net-(U4-Rs)")
+			(net 52 "RS")
 			(pinfunction "Rs")
 			(pintype "input")
@@
 	)
 	(segment
-		(start 150.9795 97.536)
-		(end 150.9795 99.1635)
-		(width 0.2)
-		(layer "F.Cu")
-		(net 50)
-	)
-	(segment
-		(start 151.2712 99.4552)
-		(end 152.335 99.4552)
-		(width 0.2)
-		(layer "F.Cu")
-		(net 50)
-	)
-	(segment
-		(start 150.9795 99.1635)
-		(end 151.2712 99.4552)
-		(width 0.2)
-		(layer "F.Cu")
-		(net 50)
-	)
-	(segment
 		(start 133.88 107.7)
 		(end 133.89 107.69)
 		(width 0.4)
 		(layer "F.Cu")
-		(net 52)
+		(net 51)
 	)
 	(segment
@@
 		(width 0.4)
 		(layer "F.Cu")
-		(net 52)
+		(net 51)
 	)
 	(segment
@@
 		(width 0.4)
 		(layer "F.Cu")
-		(net 52)
+		(net 51)
 	)
 	(segment
@@
 		(width 0.4)
 		(layer "F.Cu")
-		(net 52)
+		(net 51)
 	)
 	(segment
@@
 		(width 0.4)
 		(layer "F.Cu")
+		(net 51)
+	)
+	(segment
+		(start 150.9795 97.536)
+		(end 150.9795 99.1635)
+		(width 0.2)
+		(layer "F.Cu")
+		(net 52)
+	)
+	(segment
+		(start 151.2712 99.4552)
+		(end 152.335 99.4552)
+		(width 0.2)
+		(layer "F.Cu")
+		(net 52)
+	)
+	(segment
+		(start 150.9795 99.1635)
+		(end 151.2712 99.4552)
+		(width 0.2)
+		(layer "F.Cu")
 		(net 52)

Commit message: Ultimos cambios y revisiones
Changed lines of the file:
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@@
 		(tags "9-pin D-Sub connector horizontal angled 90deg THT pins pitch 2.77x2.54mm pin-PCB-offset 9.4mm")
 		(property "Reference" "J8"
-			(at 5.54 -1.8 0)
+			(at -2.26 0 0)
 			(layer "F.SilkS")
 			(effects
@@
 			)
 		)
+	)
+	(dimension
+		(type orthogonal)
+		(layer "F.Cu")
+		(pts
+			(xy 173.802 143.2408) (xy 108.1934 143.2408)
+		)
+		(height 6.0492)
+		(orientation 0)
+		(format
+			(prefix "")
+			(suffix "")
+			(units 3)
+			(units_format 0)
+			(precision 4)
+			(suppress_zeroes yes)
+		)
+		(style
+			(thickness 0.2)
+			(arrow_length 1.27)
+			(text_position_mode 0)
+			(arrow_direction outward)
+			(extension_height 0.58642)
+			(extension_offset 0.5)
+			(keep_text_aligned yes)
+		)
+		(gr_text "65,6086"
+			(at 140.9977 147.49 0)
+			(layer "F.Cu")
+			(effects
+				(font
+					(size 1.5 1.5)
+					(thickness 0.3)
+				)
+			)
+		)
+	)
+	(dimension
+		(type orthogonal)
+		(layer "F.Cu")
+		(pts
+			(xy 108.1934 143.2408) (xy 108.1934 83.1176)
+		)
+		(height -10.5634)
+		(orientation 1)
+		(format
+			(prefix "")
+			(suffix "")
+			(units 3)
+			(units_format 0)
+			(precision 4)
+			(suppress_zeroes yes)
+		)
+		(style
+			(thickness 0.2)
+			(arrow_length 1.27)
+			(text_position_mode 0)
+			(arrow_direction outward)
+			(extension_height 0.58642)
+			(extension_offset 0.5)
+			(keep_text_aligned yes)
+		)
+		(gr_text "60,1232"
+			(at 95.83 113.1792 90)
+			(layer "F.Cu")
+			(effects
+				(font
+					(size 1.5 1.5)
+					(thickness 0.3)
+				)
+			)
+		)
