File: Proyecto_Maletero/Proyecto_Maletero.kicad_sch (KiCad schematic)
At the start: 17 parts, among them J3 Conn_01x02, J4 Conn_01x03, J6 DE9_Pins, U1 LM1084-5.0, U3 PIC18F258-I_SO, Y1 4MHz

Commit message: Ultimos cambios y revisiones
Parts:
- removed C5: 1u, Capacitor_SMD:C_0805_2012Metric, symbol Device:C_Polarized_US
- added C5: 1u, Capacitor_SMD:C_0805_2012Metric, symbol Device:C
Connections:
- net GNDPWR: now also C5.2
- net VCC: now also C5.1
Other:
- moved on the sheet: C16, C6, C7, J4, Y1
